Commit message: Write a controller that can change the speed_mode and use pid and feedfront control.

File: qyd_work/fan_ws/src/fan_description/urdf/fan_description.urdf (robot description, URDF)
Before this commit: robot fan, 4 links, 3 joints
Links:
- link base_link: mass 100 -> 1000000; geometry collision box size=0.01 0.01 0.01; visual box size=0.01 0.01 0.01
Joints:
- joint pole2joint: axis (none) -> 0 1 0; type fixed -> continuous

Commit message: Fix some problem and add joint_state_publisher.

File: qyd_work/fan_ws/src/fan_description/urdf/fan_description.urdf (robot description, URDF)
Before this commit: robot fan, 4 links, 3 joints
Links:
- added link world, mass 0
- link base_link: mass 1000000 -> 1000
Joints:
- added joint base_to_ground: type fixed, parent world, child base_link, origin xyz=0 0 0 rpy=0 0 0
